File: PCB/MiniRoverShield.sch (KiCad schematic (older format))
At the start: 47 parts, among them J1 linetracer, J2 linetracer, J3 linetracer, J4 linetracer, J5 linetracer, J6 linetracer, P1 Arduino nano 33, P2 Arduino nano 33, P3 flightPin, P4 Nichrome, P5 Motor, P6 Motor, Q1 FDS4935A, Q2 IRFML8244TRPbF, Q3 L-51ROPT1D1, Q4 L-51ROPT1D1, SW1 Power, U1 TPS63000, U2 GYSFDMAXB, U3 BD6211F, U4 BD6211F

Commit message: 配線完了
Connections:
- net labels added: SCK
- net labels removed: CLK
- wire segments 216 -> 217
Changed lines of the file:
@@
 MISO
 Text Label 6800 1900 0    50   ~ 0
-CLK
+SCK
 Text Label 6800 1700 0    50   ~ 0
 MOSI
@@
 	6800 1900 7700 1900
 Text Label 3150 1100 0    50   ~ 0
-CS
+SCK
 Text Label 6100 1100 2    50   ~ 0
 MISO
 Text Label 6100 1200 2    50   ~ 0
 MOSI
+Text Label 6100 1700 2    50   ~ 0
+MotorR1
+Text Label 6100 1800 2    50   ~ 0
+MotorR2
 Text Label 6100 1300 2    50   ~ 0
-MotorR1
+MotorL1
 Text Label 6100 1400 2    50   ~ 0
-MotorR2
-Text Label 6100 1700 2    50   ~ 0
-MotorL1
-Text Label 6100 1800 2    50   ~ 0
 MotorL2
 Text Label 6100 2000 2    50   ~ 0
@@
 	4900 2000 6100 2000
 Wire Wire Line
+	4900 1400 6100 1400
+Wire Wire Line
+	4900 1300 6100 1300
+Wire Wire Line
+	4900 1700 6100 1700
+Wire Wire Line
 	4900 1800 6100 1800
 Wire Wire Line
-	4900 1700 6100 1700
-Wire Wire Line
-	4900 1300 6100 1300
-Wire Wire Line
-	4900 1400 6100 1400
-Wire Wire Line
 	4900 1200 6100 1200
 Wire Wire Line
@@
 Wire Wire Line
 	3150 1100 3600 1100
+Text Label 3150 2100 0    50   ~ 0
+PTr_R
 Text Label 3150 1500 0    50   ~ 0
-PTr_R
-Text Label 3150 1600 0    50   ~ 0
 RTr_L
 Wire Wire Line
 	3600 1500 3150 1500
 Wire Wire Line
-	3600 1600 3150 1600
+	3600 2100 3150 2100
 $Comp
 L user_library:TPS63000 U1
@@
 L Connector_Generic:Conn_01x02 P5
 U 1 1 5D433612
-P 8500 3850
-F 0 "P5" H 8580 3796 50  0000 L CNN
-F 1 "Motor" H 8580 3751 50  0001 L CNN
-F 2 "Connector_JST:JST_EH_B02B-EH-A_1x02_P2.50mm_Vertical" H 8500 3850 50  0001 C CNN
-F 3 "~" H 8500 3850 50  0001 C CNN
-	1    8500 3850
-	1    0    0    -1
+P 8500 3950
+F 0 "P5" H 8580 3896 50  0000 L CNN
+F 1 "Motor" H 8580 3851 50  0001 L CNN
+F 2 "Connector_JST:JST_EH_B02B-EH-A_1x02_P2.50mm_Vertical" H 8500 3950 50  0001 C CNN
+F 3 "~" H 8500 3950 50  0001 C CNN
+	1    8500 3950
+	1    0    0    1
 $EndComp
 Text Label 6500 4000 0    50   ~ 0
@@
 Wire Wire Line
 	8800 5100 9200 5100
-Text Label 6100 2100 2    50   ~ 0
+Text Label 6100 1600 2    50   ~ 0
 flightPin
 Wire Wire Line
-	6100 2100 4900 2100
+	6100 1600 4900 1600
 $Comp
 L Connector_Generic:Conn_01x02 P3
@@
 	1    0    0    -1
 $EndComp
+Text Label 6100 1500 2    50   ~ 0
+CS
+Wire Wire Line
+	4900 1500 6100 1500
 $EndSCHEMATC

Commit message: Remove Line Trace
Parts:
- removed D3, D4: OSI5LA5A33A-B, user:LED_5mm_2.54mm, symbol Device:LED
- removed J1, J2: linetracer, Connector_PinHeader_2.54mm:PinHeader_1x03_P2.54mm_Vertical, symbol Connector:Conn_01x03_Female
- removed J3, J4: linetracer, Connector_PinSocket_2.54mm:PinSocket_1x03_P2.54mm_Vertical, symbol Connector:Conn_01x03_Male
- removed J5, J6: linetracer, Connector_PinSocket_2.54mm:PinSocket_1x03_P2.54mm_Horizontal, symbol Connector:Conn_01x03_Male
- removed Q3, Q4: L-51ROPT1D1, user:LED_5mm_2.54mm, symbol Device:Q_Photo_NPN_CE
- removed R10, R11, R12, R9: 1K, Resistor_THT:R_Axial_DIN0204_L3.6mm_D1.6mm_P5.08mm_Horizontal, symbol Device:R_Small
- Q1, U3, U4: footprint Package_SO:SO-8_5.3x6.2mm_P1.27mm -> Package_SO:SOIC-8_3.9x4.9mm_P1.27mm
- renumbered P3 to J1, P5 to M1, P6 to M2, P4 to N1, U2 to P3, R6 to R5, R7 to R6, R8 to R7, R5 to R8
Connections:
- net labels removed: PTr_R, RTr_L
- wire segments 217 -> 173
