File: PCB/MiniRoverShield.sch (KiCad schematic (older format))
At the start: 33 parts, among them J1 flightPin, M1 Motor, M2 Motor, P1 Arduino nano 33, P2 Arduino nano 33, P3 GYSFDMAXB, Q1 FDS4935A, Q2 IRFML8244TRPbF, SW1 Power, U1 TPS63000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

Commit message: Update MiniRoverShield.sch
Parts:
- U1: value TPS63000 -> TPS63001
Changed lines of the file:
@@
 P 1450 3000
 F 0 "U1" H 1450 3667 50  0000 C CNN
-F 1 "TPS63000" H 1450 3576 50  0000 C CNN
+F 1 "TPS63001" H 1450 3576 50  0000 C CNN
 F 2 "Package_SON:Texas_S-PVSON-N10_ThermalVias" H 1450 2350 50  0001 C CNN
 F 3 "https://strawberry-linux.com/pub/tps63000.pdf" H 1450 3000 50  0001 C CNN
